File: pcb/SilentStepStick_v10.brd (EAGLE design)
At the start: 15.2 x 20.3 mm, 30 parts, among them X1 PASSER-07, X2 PASSER-07

Commit message: updated layout and schematics
Parts:
- CFG1, CFG2, CFG3, CFG6: value JUMPER2-0201-NC -> JUMPER2-0201; device we-rcl:JUMPER2-0201_NC -> we-rcl:JUMPER2-0201
- CFG5: value JUMPER3-0201-NC -> JUMPER3-0201; device we-rcl:JUMPER3-0201_NC -> we-rcl:JUMPER3-0201
Changed lines of the file:
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@@
 <setting verticaltext="up"/>
 </settings>
-<grid distance="0.05" unitdist="inch" unit="inch" style="lines" multiple="1" display="yes" altdistance="0.0125" altunitdist="inch" altunit="inch"/>
+<grid distance="0.05" unitdist="inch" unit="inch" style="lines" multiple="1" display="yes" altdistance="0.025" altunitdist="inch" altunit="inch"/>
 <layers>
 <layer number="1" name="Top" color="4" fill="1" visible="yes" active="yes"/>
@@
 <text x="8.935" y="4.064" size="1" layer="22" font="vector" ratio="14" rot="MR90">SilentStepStick</text>
 <text x="3.048" y="20.273" size="0.6858" layer="22" font="vector" ratio="13" rot="MR180">www.watterott.com</text>
-<rectangle x1="2.7686" y1="2.7686" x2="3.0734" y2="3.2004" layer="31"/>
-<rectangle x1="3.2766" y1="2.7686" x2="3.5814" y2="3.2004" layer="31"/>
-<rectangle x1="9.7536" y1="8.0518" x2="10.0584" y2="8.4836" layer="31"/>
-<rectangle x1="10.2616" y1="8.0518" x2="10.5664" y2="8.4836" layer="31"/>
-<rectangle x1="10.7696" y1="8.0518" x2="11.0744" y2="8.4836" layer="31"/>
-<rectangle x1="2.7686" y1="6.1214" x2="3.0734" y2="6.5532" layer="31"/>
-<rectangle x1="3.2766" y1="6.1214" x2="3.5814" y2="6.5532" layer="31"/>
-<rectangle x1="2.7686" y1="8.6614" x2="3.0734" y2="9.0932" layer="31"/>
-<rectangle x1="3.2766" y1="8.6614" x2="3.5814" y2="9.0932" layer="31"/>
 </plain>
 <attributes>
@@
 <attribute name="NAME" x="10.457" y="17.6" size="0.4064" layer="25" font="vector" ratio="10"/>
 </element>
-<element name="CFG3" library="we-rcl" package="JUMPER2-0201_NC" value="JUMPER2-0201-NC" x="3.175" y="8.89" smashed="yes" rot="R270">
+<element name="CFG3" library="we-rcl" package="JUMPER2-0201" value="JUMPER2-0201" x="3.175" y="8.89" smashed="yes" rot="R270">
 <attribute name="NAME" x="3.6125" y="8.154" size="0.4064" layer="25" font="vector" ratio="10" align="center"/>
 </element>
@@
 <attribute name="NAME" x="11.4765" y="5.1695" size="0.4064" layer="25" font="vector" ratio="10" align="center"/>
 </element>
-<element name="CFG5" library="we-rcl" package="JUMPER3-0201_NC" value="JUMPER3-0201-NC" x="10.414" y="8.255" smashed="yes" rot="R270">
+<element name="CFG5" library="we-rcl" package="JUMPER3-0201" value="JUMPER3-0201" x="10.414" y="8.255" smashed="yes" rot="R270">
 <attribute name="NAME" x="10.414" y="9.019" size="0.4064" layer="25" font="vector" ratio="10" align="center"/>
 </element>
-<element name="CFG6" library="we-rcl" package="JUMPER2-0201_NC" value="JUMPER2-0201-NC" x="3.175" y="2.9845" smashed="yes" rot="R270">
+<element name="CFG6" library="we-rcl" package="JUMPER2-0201" value="JUMPER2-0201" x="3.175" y="2.9845" smashed="yes" rot="R270">
 <attribute name="NAME" x="3.175" y="2.2485" size="0.4064" layer="25" font="vector" ratio="10" align="center"/>
 </element>
-<element name="CFG1" library="we-rcl" package="JUMPER2-0201_NC" value="JUMPER2-0201-NC" x="3.175" y="3.81" smashed="yes" rot="R270">
+<element name="CFG1" library="we-rcl" package="JUMPER2-0201" value="JUMPER2-0201" x="3.175" y="3.81" smashed="yes" rot="R270">
 <attribute name="NAME" x="3.4875" y="4.5115" size="0.4064" layer="25" font="vector" ratio="10" align="center"/>
 </element>
-<element name="CFG2" library="we-rcl" package="JUMPER2-0201_NC" value="JUMPER2-0201-NC" x="3.175" y="6.35" smashed="yes" rot="R270">
+<element name="CFG2" library="we-rcl" package="JUMPER2-0201" value="JUMPER2-0201" x="3.175" y="6.35" smashed="yes" rot="R270">
 <attribute name="NAME" x="3.925" y="7.0515" size="0.4064" layer="25" font="vector" ratio="10" align="center"/>
 </element>
@@
 <via x="10.922" y="7.747" extent="1-16" drill="0.3"/>
 <wire x1="10.922" y1="7.747" x2="10.922" y2="8.254" width="0.16" layer="1"/>
-<wire x1="10.922" y1="8.254" x2="10.923" y2="8.255" width="0.16" layer="1"/>
+<wire x1="10.922" y1="8.254" x2="10.924" y2="8.255" width="0.16" layer="1"/>
 <via x="3.4395" y="14.996" extent="1-16" drill="0.3"/>
 <via x="11.684" y="19.685" extent="1-16" drill="0.3"/>
@@
 <wire x1="9.905" y1="5.9055" x2="9.906" y2="5.9045" width="0.16" layer="1"/>
 <wire x1="9.906" y1="8.3175" x2="9.905" y2="8.3165" width="0.16" layer="1"/>
-<wire x1="9.905" y1="8.3165" x2="9.905" y2="8.255" width="0.16" layer="1"/>
+<wire x1="9.905" y1="8.3165" x2="9.904" y2="8.255" width="0.16" layer="1"/>
 <wire x1="10.7875" y1="12.6875" x2="10.7875" y2="11.1835" width="0.16" layer="1"/>
 <wire x1="10.7875" y1="11.1835" x2="11.43" y2="10.541" width="0.16" layer="1"/>
@@
 <wire x1="9.554" y1="9.75" x2="10.414" y2="8.89" width="0.16" layer="1"/>
 <wire x1="10.414" y1="8.89" x2="10.414" y2="8.256" width="0.16" layer="1"/>
-<wire x1="10.414" y1="8.256" x2="10.413" y2="8.255" width="0.16" layer="1"/>
+<wire x1="10.414" y1="8.256" x2="10.414" y2="8.255" width="0.16" layer="1"/>
 </signal>
 <signal name="CFG4">

Commit message: updated schematics
Parts:
- R2, R4: value R0805/0R27 -> R0805/0R11
- R6: value (none) -> 20k
- renumbered U$1 to IC1
Changed lines of the file:
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@@
 </autorouter>
 <elements>
-<element name="U$1" library="TMC2100_QFN" package="QFN36" value="TMC2100_QFN36" x="6.75" y="12" smashed="yes"/>
+<element name="IC1" library="TMC2100_QFN" package="QFN36" value="TMC2100_QFN36" x="6.75" y="12" smashed="yes"/>
 <element name="JP1" library="pinhead-2" package="1X08-S" value="" x="1.27" y="10.16" smashed="yes" rot="R270">
 <attribute name="VALUE" x="-1.905" y="20.32" size="1.27" layer="27" rot="R270"/>
@@
 <attribute name="NAME" x="7.8735" y="6.254" size="0.4064" layer="25" font="vector" ratio="10"/>
 </element>
-<element name="R2" library="rcl" package="M0805" value="R0805/0R27" x="6.125" y="6.25" smashed="yes" rot="R90">
+<element name="R2" library="rcl" package="M0805" value="R0805/0R11" x="6.125" y="6.25" smashed="yes" rot="R90">
 <attribute name="NAME" x="5.165" y="6.0975" size="0.4064" layer="25" font="vector" ratio="10" rot="R90"/>
 </element>
-<element name="R4" library="rcl" package="M0805" value="R0805/0R27" x="6.25" y="17.8125" smashed="yes" rot="R270">
+<element name="R4" library="rcl" package="M0805" value="R0805/0R11" x="6.25" y="17.8125" smashed="yes" rot="R270">
 <attribute name="NAME" x="5.3075" y="15.5875" size="0.4064" layer="25" font="vector" ratio="10"/>
 </element>
@@
 <attribute name="NAME" x="11.3925" y="6.6647" size="0.4064" layer="25" font="vector" ratio="10"/>
 </element>
-<element name="R6" library="we-rcl" package="POT_EVM3R" value="" x="10.033" y="1.8415" smashed="yes" rot="R90">
+<element name="R6" library="we-rcl" package="POT_EVM3R" value="20k" x="10.033" y="1.8415" smashed="yes" rot="R90">
 <attribute name="NAME" x="10.033" y="0.62" size="0.4064" layer="25" font="vector" ratio="10" rot="R180" align="center"/>
 <attribute name="VALUE" x="10.033" y="4.0005" size="0.8128" layer="27" font="vector" ratio="10" rot="R180" align="center"/>
@@
 <signals>
 <signal name="CFG6">
-<contactref element="U$1" pad="22"/>
+<contactref element="IC1" pad="22"/>
 <contactref element="CFG6" pad="1"/>
 <wire x1="9.525" y1="11.2395" x2="12.1285" y2="8.636" width="0.16" layer="1"/>
@@
 </signal>
 <signal name="CFG1">
-<contactref element="U$1" pad="4"/>
+<contactref element="IC1" pad="4"/>
 <contactref element="CFG1" pad="1"/>
 <wire x1="4.35" y1="12.75" x2="3.86" y2="12.75" width="0.18" layer="1"/>
@@
 </signal>
 <signal name="CFG2">
-<contactref element="U$1" pad="3"/>
+<contactref element="IC1" pad="3"/>
 <contactref element="CFG2" pad="1"/>
 <wire x1="4.35" y1="13.25" x2="3.598" y2="13.25" width="0.18" layer="1"/>
@@
 </signal>
 <signal name="CFG3">
-<contactref element="U$1" pad="2"/>
+<contactref element="IC1" pad="2"/>
 <contactref element="CFG3" pad="1"/>
 <wire x1="4.35" y1="13.75" x2="3.776" y2="13.75" width="0.18" layer="1"/>
@@
 </signal>
 <signal name="DIAG0">
-<contactref element="U$1" pad="20"/>
+<contactref element="IC1" pad="20"/>
 <wire x1="9.15" y1="10.25" x2="9.6255" y2="10.25" width="0.16" layer="1"/>
 <wire x1="9.6255" y1="10.25" x2="11.4935" y2="8.382" width="0.16" layer="1"/>
@@
 </signal>
 <signal name="DIAG1">
-<contactref element="U$1" pad="21"/>
+<contactref element="IC1" pad="21"/>
 <wire x1="9.15" y1="10.75" x2="9.57" y2="10.75" width="0.16" layer="1"/>
 <wire x1="9.57" y1="10.75" x2="11.811" y2="8.509" width="0.16" layer="1"/>
@@
 <signal name="STEP">
 <contactref element="JP1" pad="2"/>
-<contactref element="U$1" pad="6"/>
+<contactref element="IC1" pad="6"/>
 <wire x1="4.35" y1="11.75" x2="2.982" y2="11.75" width="0.18" layer="1"/>
 <wire x1="2.982" y1="11.75" x2="2.794" y2="11.938" width="0.18" layer="1"/>
@@
 <signal name="DIR">
 <contactref element="JP1" pad="1"/>
-<contactref element="U$1" pad="7"/>
+<contactref element="IC1" pad="7"/>
 <wire x1="4.35" y1="11.25" x2="2.847" y2="11.25" width="0.18" layer="1"/>
 <wire x1="2.847" y1="11.25" x2="2.413" y2="11.684" width="0.18" layer="1"/>
@@
 <signal name="VM">
 <contactref element="JP2" pad="1"/>
-<contactref element="U$1" pad="30"/>
+<contactref element="IC1" pad="30"/>
 <contactref element="C1" pad="2"/>
-<contactref element="U$1" pad="16"/>
-<contactref element="U$1" pad="31"/>
+<contactref element="IC1" pad="16"/>
+<contactref element="IC1" pad="31"/>
 <contactref element="C6" pad="2"/>
 <contactref element="C7" pad="2"/>
@@
 <contactref element="JP2" pad="2"/>
 <contactref element="JP2" pad="8"/>
-<contactref element="U$1" pad="10"/>
+<contactref element="IC1" pad="10"/>
 <contactref element="C1" pad="1"/>
-<contactref element="U$1" pad="24"/>
-<contactref element="U$1" pad="GND_PAD"/>
-<contactref element="U$1" pad="11"/>
-<contactref element="U$1" pad="35"/>
-<contactref element="U$1" pad="12"/>
+<contactref element="IC1" pad="24"/>
+<contactref element="IC1" pad="GND_PAD"/>
+<contactref element="IC1" pad="11"/>
+<contactref element="IC1" pad="35"/>
+<contactref element="IC1" pad="12"/>
 <contactref element="C4" pad="2"/>
 <contactref element="C3" pad="2"/>
 <contactref element="C2" pad="2"/>
 <contactref element="C7" pad="1"/>
-<contactref element="U$1" pad="1"/>
+<contactref element="IC1" pad="1"/>
 <contactref element="R2" pad="1"/>
 <contactref element="R4" pad="1"/>
-<contactref element="U$1" pad="36"/>
+<contactref element="IC1" pad="36"/>
 <polygon width="0.2" layer="1" rank="6">
 <vertex x="0" y="20.32"/>
@@
 <contactref element="CFG4" pad="1"/>
 <contactref element="CFG5" pad="1"/>
-<contactref element="U$1" pad="5"/>
+<contactref element="IC1" pad="5"/>
 <wire x1="4.35" y1="12.25" x2="5.375" y2="12.25" width="0.18" layer="1"/>
 <wire x1="5.375" y1="12.25" x2="5.625" y2="12" width="0.18" layer="1"/>
@@
 </signal>
 <signal name="OA1">
-<contactref element="U$1" pad="34"/>
+<contactref element="IC1" pad="34"/>
 <polygon width="0.2" layer="1" thermals="no" rank="2">
 <vertex x="6.25" y="14.625"/>
@@
 </signal>
 <signal name="OA2">
-<contactref element="U$1" pad="32"/>
+<contactref element="IC1" pad="32"/>
 <polygon width="0.2" layer="1" thermals="no" rank="3">
 <vertex x="8.125" y="14.625"/>
@@
 </signal>
 <signal name="OB2">
-<contactref element="U$1" pad="15"/>
+<contactref element="IC1" pad="15"/>
 <polygon width="0.2" layer="1" thermals="no" rank="3">
 <vertex x="8.25" y="6.4425"/>
@@
 </signal>
 <signal name="OB1">
-<contactref element="U$1" pad="13"/>
+<contactref element="IC1" pad="13"/>
 <polygon width="0.2" layer="1" thermals="no" rank="2">
 <vertex x="6.3125" y="7.141"/>
@@
 <contactref element="JP2" pad="7"/>
 <contactref element="C2" pad="1"/>
-<contactref element="U$1" pad="8"/>
+<contactref element="IC1" pad="8"/>
 <polygon width="0.2" layer="15">
 <vertex x="15.24" y="15.359"/>
@@
 </signal>
 <signal name="VCC">
-<contactref element="U$1" pad="26"/>
+<contactref element="IC1" pad="26"/>
 <contactref element="C3" pad="1"/>
 <contactref element="R1" pad="2"/>
@@
 </signal>
 <signal name="VCP">
-<contactref element="U$1" pad="29"/>
+<contactref element="IC1" pad="29"/>
 <contactref element="C6" pad="1"/>
 <wire x1="8.5" y1="14.9" x2="9.775" y2="14.9" width="0.254" layer="1"/>
@@
 </signal>
 <signal name="CPI">
-<contactref element="U$1" pad="28"/>
+<contactref element="IC1" pad="28"/>
 <contactref element="C5" pad="1"/>
 <wire x1="9.15" y1="14.25" x2="9.75" y2="14.25" width="0.254" layer="1"/>
@@
 </signal>
 <signal name="CPO">
-<contactref element="U$1" pad="27"/>
+<contactref element="IC1" pad="27"/>
 <contactref element="C5" pad="2"/>
 <wire x1="9.15" y1="13.75" x2="9.875" y2="13.75" width="0.254" layer="1"/>
@@
 </signal>
 <signal name="N$7">
-<contactref element="U$1" pad="33"/>
+<contactref element="IC1" pad="33"/>
 <contactref element="R4" pad="2"/>
 <wire x1="6.5" y1="14.9" x2="6.5" y2="16.6125" width="0.254" layer="1"/>
@@
 </signal>
 <signal name="N$9">
-<contactref element="U$1" pad="14"/>
+<contactref element="IC1" pad="14"/>
 <contactref element="R2" pad="2"/>
 <wire x1="6.5" y1="9.1" x2="6.5" y2="7.575" width="0.254" layer="1"/>
@@
 <signal name="+5V">
 <contactref element="C4" pad="1"/>
-<contactref element="U$1" pad="25"/>
+<contactref element="IC1" pad="25"/>
 <contactref element="R1" pad="1"/>
 <wire x1="9.15" y1="12.75" x2="10.7875" y2="12.75" width="0.254" layer="1"/>
@@
 </signal>
 <signal name="CFG5">
-<contactref element="U$1" pad="19"/>
+<contactref element="IC1" pad="19"/>
 <contactref element="CFG5" pad="2"/>
 <wire x1="9.15" y1="9.75" x2="9.554" y2="9.75" width="0.16" layer="1"/>
@@
 </signal>
 <signal name="CFG4">
-<contactref element="U$1" pad="18"/>
+<contactref element="IC1" pad="18"/>
 <contactref element="R3" pad="2"/>
 <wire x1="8.5" y1="9.1" x2="9.398" y2="8.202" width="0.16" layer="1"/>
@@
 </signal>
 <signal name="IREF">
-<contactref element="U$1" pad="23"/>
+<contactref element="IC1" pad="23"/>
 <wire x1="9.47" y1="11.7475" x2="9.1525" y2="11.7475" width="0.16" layer="1"/>
 <wire x1="9.1525" y1="11.7475" x2="9.15" y2="11.75" width="0.16" layer="1"/>
