File: pcb/SilentStepStick_v11.brd (EAGLE design)
At the start: 15.2 x 20.3 mm, 30 parts, among them IC1 TMC2100_QFN36, X1 PASSER-07, X2 PASSER-07

Commit message: updated layout and schematics
Parts:
- removed R3: R0402/0, rcl:R0402
- added CFG0: JUMPER3-0201, we-rcl:JUMPER3-0201
- C1, C2, C6, C7: value C0402/100nF/50V -> 100n/50V; device rcl:C0402 -> we-rcl:R0402
- C3: value C0402/470nF/10V -> 470n/10V; device rcl:C0402 -> we-rcl:R0402
- C4: value C0402/4.7uF/10V -> 4u7/10V; device rcl:C0402 -> we-rcl:R0402
- C5: value C0402/22nF/50V -> 22n/50V; device rcl:C0402 -> we-rcl:R0402
- CFG4: value JUMPER3-0201-NC -> JUMPER3-0201; device we-rcl:JUMPER3-0201_NC -> we-rcl:JUMPER3-0201
- R1: value R0402/2R2 -> 2R2; device rcl:R0402 -> we-rcl:R0402
- R5: value R0402/20k -> 20k; device rcl:R0402 -> we-rcl:R0402
- moved C2 8.89 mm to (12.2, 17.0), turned to 0 degrees
- moved CFG5 1.11 mm to (10.4, 7.14), turned to 90 degrees
- moved C6 0.62 mm to (10.3, 17.4), turned to 90 degrees
- moved C7 0.48 mm to (8.57, 6.10)
- moved IC1 0.25 mm to (7.00, 12.0)
- moved R1 0.20 mm to (11.9, 11.2), turned to 0 degrees
- moved C5 0.17 mm to (10.8, 14.6), turned to 180 degrees
- moved C3 0.16 mm to (11.9, 14.6), turned to 0 degrees
- moved C4 0.14 mm to (11.3, 12.7), turned to 270 degrees
- moved C1 0.10 mm to (8.76, 18.0), turned to 180 degrees
- moved CFG4 0.10 mm to (10.4, 6.00), turned to 90 degrees
- moved R5 0.07 mm to (8.76, 4.57), turned to 90 degrees
Connections:
- removed net N$1: CFG4.2, R3.1
- new net CFG0: CFG0.2, IC1.5
- net +5V: now also C4.2, R1.2; no longer C4.1, CFG4.3, CFG5.3, R1.1
- net CFG4: now also CFG4.2; no longer R3.2
- net CPI: now also C5.2; no longer C5.1
- net CPO: now also C5.1; no longer C5.2
- net GND: now also C1.2, C2.1, C3.1, C4.1, C7.2, CFG0.1; no longer C1.1, C2.2, C3.2, C4.2, C7.1, IC1.5
- net VCC: now also C3.2, R1.1; no longer C3.1, R1.2
- net VCP: now also C6.2; no longer C6.1
- net VIO: now also C2.2, CFG0.3, CFG4.3, CFG5.3; no longer C2.1
- net VM: now also C1.1, C6.1, C7.1; no longer C1.2, C6.2, C7.2
Routing:
- net VIO: track 1.82 -> 14.8 mm, vias 2 -> 3
- net CFG0: track 0.00 -> 8.81 mm, vias 0 -> 2
- net +5V: track 20.7 -> 16.1 mm
- net GND: track 5.07 -> 2.50 mm, vias 40 -> 36
- net CFG4: track 2.67 -> 5.24 mm
- net VM: track 5.66 -> 3.28 mm, vias 4 -> 3
- net CFG3: track 9.45 -> 11.3 mm
- net CFG2: track 8.81 -> 10.5 mm
- net N$1: track 1.70 -> 0.00 mm
- net CFG1: track 10.1 -> 11.2 mm
- net VCP: track 4.68 -> 3.73 mm
- net CFG5: track 2.26 -> 3.11 mm
- net CPI: track 2.51 -> 1.77 mm
- net N$10: track 0.51 -> 0.00 mm
Other:
- board text added: "TOP"
