File: pcb/SilentStepStick_v11.sch (EAGLE design)
At the start: 30 parts, among them IC1 TMC2100_QFN36, X1 PASSER-07, X2 PASSER-07

Commit message: updated layout and schematics
Parts:
- removed R3: R0402/0, rcl:R-EU_R0402
- added CFG0: JUMPER3-0201, we-rcl:JUMPER3-0201
- C1, C2, C6, C7: value C0402/100nF/50V -> 100n/50V; device rcl:C-EUC0402 -> we-rcl:CAPACITOR-C0402
- C3: value C0402/470nF/10V -> 470n/10V; device rcl:C-EUC0402 -> we-rcl:CAPACITOR-C0402
- C4: value C0402/4.7uF/10V -> 4u7/10V; device rcl:C-EUC0402 -> we-rcl:CAPACITOR-C0402
- C5: value C0402/22nF/50V -> 22n/50V; device rcl:C-EUC0402 -> we-rcl:CAPACITOR-C0402
- CFG4: value JUMPER3-0201-NC -> JUMPER3-0201; device we-rcl:JUMPER3-0201-NC -> we-rcl:JUMPER3-0201
- R1: value R0402/2R2 -> 2R2; device rcl:R-EU_R0402 -> we-rcl:RESISTOR-R0402
- R5: value R0402/20k -> 20k; device rcl:R-EU_R0402 -> we-rcl:RESISTOR-R0402
Connections:
- removed net N$1: CFG4.2, R3.1
- new net CFG0: CFG0.2, IC1.SDO_NAO_CFG0
- net +5V: now also C4.2, R1.2; no longer C4.1, CFG4.3, CFG5.3, R1.1
- net CFG4: now also CFG4.2; no longer R3.2
- net CPI: now also C5.2; no longer C5.1
- net CPO: now also C5.1; no longer C5.2
- net GND: now also C1.2, C2.1, C3.1, C4.1, C7.2, CFG0.1; no longer C1.1, C2.2, C3.2, C4.2, C7.1, IC1.SDO_NAO_CFG0
- net VCC: now also C3.2, R1.1; no longer C3.1, R1.2
- net VCP: now also C6.2; no longer C6.1
- net VIO: now also C2.2, CFG0.3, CFG4.3, CFG5.3; no longer C2.1
- net VM: now also C1.1, C6.1, C7.1; no longer C1.2, C6.2, C7.2
Other:
- moved on the sheet: CFG4, CFG5, CFG6
