File: hardware/SilentStepStick_v12.brd (EAGLE design)
At the start: 15.2 x 20.3 mm, 30 parts, among them IC1 TMC2100_QFN36, X1 PASSER-07, X2 PASSER-07

Commit message: updated layout and schematics
Parts:
- C8: value C0603/1uF/50V -> 1u/50V
- IC1: value TMC2100_QFN36 -> TMC2100-LA; device TMC2100_QFN:QFN36 -> we-chip:QFN36-PAD
Connections:
- net N$7 renamed BRA
- net N$9 renamed BRB
- net GND: now also IC1.TP; no longer IC1.GND_PAD
Routing:
- net GND: track 4.42 -> 6.63 mm
